File: schematics/STM32L052_Breakout.sch (EAGLE design)
At the start: 0 parts

Commit message: more libraries and datasheets
Parts:
- added MCU: STM32L052K8T, STM32L052:MICRO-STM_V3_STM32L052K8T
- added R1: 10k, SparkFun-Resistors:10KOHM-0603-1/10W-1%
Connections:
- new net GND: R1.1
- new net N$1: MCUMCU.BOOT0, R1.2
Changed lines of the file:
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@@
 <layer number="48" name="Document" color="7" fill="1" visible="no" active="no"/>
 <layer number="49" name="Reference" color="7" fill="1" visible="no" active="no"/>
+<layer number="50" name="dxf" color="7" fill="1" visible="no" active="no"/>
 <layer number="51" name="tDocu" color="7" fill="1" visible="no" active="no"/>
 <layer number="52" name="bDocu" color="7" fill="1" visible="no" active="no"/>
+<layer number="53" name="tGND_GNDA" color="7" fill="1" visible="no" active="no"/>
+<layer number="54" name="bGND_GNDA" color="7" fill="1" visible="no" active="no"/>
+<layer number="56" name="wert" color="7" fill="1" visible="no" active="no"/>
+<layer number="57" name="tCAD" color="7" fill="1" visible="no" active="no"/>
+<layer number="59" name="tCarbon" color="7" fill="1" visible="no" active="no"/>
+<layer number="60" name="bCarbon" color="7" fill="1" visible="no" active="no"/>
 <layer number="88" name="SimResults" color="9" fill="1" visible="yes" active="yes"/>
 <layer number="89" name="SimProbes" color="9" fill="1" visible="yes" active="yes"/>
@@
 <layer number="97" name="Info" color="7" fill="1" visible="yes" active="yes"/>
 <layer number="98" name="Guide" color="6" fill="1" visible="yes" active="yes"/>
+<layer number="99" name="SpiceOrder" color="7" fill="1" visible="yes" active="yes"/>
+<layer number="100" name="Muster" color="7" fill="1" visible="yes" active="yes"/>
+<layer number="101" name="Patch_Top" color="7" fill="1" visible="yes" active="yes"/>
+<layer number="102" name="Vscore" color="7" fill="1" visible="yes" active="yes"/>
+<layer number="103" name="tMap" color="7" fill="1" visible="yes" active="yes"/>
+<layer number="104" name="Name" color="7" fill="1" visible="yes" active="yes"/>
+<layer number="105" name="tPlate" color="7" fill="1" visible="yes" active="yes"/>
+<layer number="106" name="bPlate" color="7" fill="1" visible="yes" active="yes"/>
+<layer number="107" name="Crop" color="7" fill="1" visible="yes" active="yes"/>
+<layer number="108" name="tplace-old" color="7" fill="1" visible="yes" active="yes"/>
+<layer number="109" name="ref-old" color="7" fill="1" visible="yes" active="yes"/>
+<layer number="110" name="fp0" color="7" fill="1" visible="yes" active="yes"/>
+<layer number="111" name="LPC17xx" color="7" fill="1" visible="yes" active="yes"/>
+<layer number="112" name="tSilk" color="7" fill="1" visible="yes" active="yes"/>
+<layer number="113" name="IDFDebug" color="7" fill="1" visible="yes" active="yes"/>
+<layer number="114" name="Badge_Outline" color="7" fill="1" visible="yes" active="yes"/>
+<layer number="115" name="ReferenceISLANDS" color="7" fill="1" visible="yes" active="yes"/>
+<layer number="116" name="Patch_BOT" color="7" fill="1" visible="yes" active="yes"/>
+<layer number="118" name="Rect_Pads" color="7" fill="1" visible="yes" active="yes"/>
+<layer number="121" name="_tsilk" color="7" fill="1" visible="yes" active="yes"/>
+<layer number="122" name="_bsilk" color="7" fill="1" visible="yes" active="yes"/>
+<layer number="123" name="tTestmark" color="7" fill="1" visible="yes" active="yes"/>
+<layer number="124" name="bTestmark" color="7" fill="1" visible="yes" active="yes"/>
+<layer number="125" name="_tNames" color="7" fill="1" visible="yes" active="yes"/>
+<layer number="126" name="_bNames" color="7" fill="1" visible="yes" active="yes"/>
+<layer number="127" name="_tValues" color="7" fill="1" visible="yes" active="yes"/>
+<layer number="128" name="_bValues" color="7" fill="1" visible="yes" active="yes"/>
+<layer number="129" name="Mask" color="7" fill="1" visible="yes" active="yes"/>
+<layer number="131" name="tAdjust" color="7" fill="1" visible="yes" active="yes"/>
+<layer number="132" name="bAdjust" color="7" fill="1" visible="yes" active="yes"/>
+<layer number="144" name="Drill_legend" color="7" fill="1" visible="yes" active="yes"/>
+<layer number="150" name="Notes" color="7" fill="1" visible="yes" active="yes"/>
+<layer number="151" name="HeatSink" color="7" fill="1" visible="yes" active="yes"/>
+<layer number="152" name="_bDocu" color="7" fill="1" visible="yes" active="yes"/>
+<layer number="153" name="FabDoc1" color="7" fill="1" visible="yes" active="yes"/>
+<layer number="154" name="FabDoc2" color="7" fill="1" visible="yes" active="yes"/>
+<layer number="155" name="FabDoc3" color="7" fill="1" visible="yes" active="yes"/>
+<layer number="199" name="Contour" color="7" fill="1" visible="yes" active="yes"/>
+<layer number="200" name="200bmp" color="7" fill="1" visible="yes" active="yes"/>
+<layer number="201" name="201bmp" color="7" fill="1" visible="yes" active="yes"/>
+<layer number="202" name="202bmp" color="7" fill="1" visible="yes" active="yes"/>
+<layer number="203" name="203bmp" color="7" fill="1" visible="yes" active="yes"/>
+<layer number="204" name="204bmp" color="7" fill="1" visible="yes" active="yes"/>
+<layer number="205" name="205bmp" color="7" fill="1" visible="yes" active="yes"/>
+<layer number="206" name="206bmp" color="7" fill="1" visible="yes" active="yes"/>
+<layer number="207" name="207bmp" color="7" fill="1" visible="yes" active="yes"/>
+<layer number="208" name="208bmp" color="7" fill="1" visible="yes" active="yes"/>
+<layer number="209" name="209bmp" color="7" fill="1" visible="yes" active="yes"/>
+<layer number="210" name="210bmp" color="7" fill="1" visible="yes" active="yes"/>
+<layer number="211" name="211bmp" color="7" fill="1" visible="yes" active="yes"/>
+<layer number="212" name="212bmp" color="7" fill="1" visible="yes" active="yes"/>
+<layer number="213" name="213bmp" color="7" fill="1" visible="yes" active="yes"/>
+<layer number="214" name="214bmp" color="7" fill="1" visible="yes" active="yes"/>
+<layer number="215" name="215bmp" color="7" fill="1" visible="yes" active="yes"/>
+<layer number="216" name="216bmp" color="7" fill="1" visible="yes" active="yes"/>
+<layer number="217" name="217bmp" color="7" fill="1" visible="yes" active="yes"/>
+<layer number="218" name="218bmp" color="7" fill="1" visible="yes" active="yes"/>
+<layer number="219" name="219bmp" color="7" fill="1" visible="yes" active="yes"/>
+<layer number="220" name="220bmp" color="7" fill="1" visible="yes" active="yes"/>
+<layer number="221" name="221bmp" color="7" fill="1" visible="yes" active="yes"/>
+<layer number="222" name="222bmp" color="7" fill="1" visible="yes" active="yes"/>
+<layer number="223" name="223bmp" color="7" fill="1" visible="yes" active="yes"/>
+<layer number="224" name="224bmp" color="7" fill="1" visible="yes" active="yes"/>
+<layer number="225" name="225bmp" color="7" fill="1" visible="yes" active="yes"/>
+<layer number="226" name="226bmp" color="7" fill="1" visible="yes" active="yes"/>
+<layer number="227" name="227bmp" color="7" fill="1" visible="yes" active="yes"/>
+<layer number="228" name="228bmp" color="7" fill="1" visible="yes" active="yes"/>
+<layer number="229" name="229bmp" color="7" fill="1" visible="yes" active="yes"/>
+<layer number="230" name="230bmp" color="7" fill="1" visible="yes" active="yes"/>
+<layer number="231" name="231bmp" color="7" fill="1" visible="yes" active="yes"/>
+<layer number="248" name="Housing" color="7" fill="1" visible="yes" active="yes"/>
+<layer number="249" name="Edge" color="7" fill="1" visible="yes" active="yes"/>
+<layer number="250" name="Descript" color="7" fill="1" visible="yes" active="yes"/>
+<layer number="251" name="SMDround" color="7" fill="1" visible="yes" active="yes"/>
+<layer number="254" name="cooling" color="7" fill="1" visible="yes" active="yes"/>
+<layer number="255" name="routoute" color="7" fill="1" visible="yes" active="yes"/>
 </layers>
 <schematic xreflabel="%F%N/%S.%C%R" xrefpart="/%S.%C%R">
@@
 <attribute name="REV" value="1.0.0"/>
 </part>
+<part name="MCU" library="STM32L052" deviceset="MICRO-STM_V3_STM32L052K*T" device="" technology="8" value="STM32L052K8T"/>
+<part name="R1" library="SparkFun-Resistors" deviceset="10KOHM" device="-0603-1/10W-1%" package3d_urn="urn:adsk.eagle:package:39650/1" value="10k"/>
+<part name="GND1" library="Supply-Symbols" deviceset="GND" device=""/>
 </parts>
 <sheets>
@@
 <attribute name="REV" x="172.72" y="0" size="1.778" layer="96" display="off"/>
 </instance>
+<instance part="MCU" gate="MCU" x="137.16" y="116.84"/>
+<instance part="R1" gate="G$1" x="106.68" y="83.82"/>
+<instance part="GND1" gate="1" x="99.06" y="76.2"/>
 </instances>
 <busses>
 </busses>
 <nets>
+<net name="N$1" class="0">
+<segment>
+<pinref part="MCU" gate="MCU" pin="BOOT0"/>
+<pinref part="R1" gate="G$1" pin="2"/>
+<wire x1="114.3" y1="83.82" x2="111.76" y2="83.82" width="0.1524" layer="91"/>
+</segment>
+</net>
+<net name="GND" class="0">
+<segment>
+<pinref part="GND1" gate="1" pin="GND"/>
+<pinref part="R1" gate="G$1" pin="1"/>
+<wire x1="99.06" y1="78.74" x2="99.06" y2="83.82" width="0.1524" layer="91"/>
+<wire x1="99.06" y1="83.82" x2="101.6" y2="83.82" width="0.1524" layer="91"/>
+</segment>
+</net>
 </nets>
 </sheet>
@@
 will not be understood (or retained) with this version.
 </note>
+<note version="8.3" severity="warning">
+Since Version 8.3, EAGLE supports the association of 3D packages
+with devices in libraries, schematics, and board files. Those 3D
+packages will not be understood (or retained) with this version.
+</note>
 </compatibility>

Commit message: breakout progress
Parts:
- added C1, C2: 10nF, SparkFun-Capacitors:10NF-0603-50V-10%
- added C3, C6: 10uF, SparkFun-Capacitors:10UF-0603-6.3V-20%
- added C4, C5, C7: 0.1uF, SparkFun-Capacitors:0.1UF-0603-25V-(+80/-20%)
- added J1: Breakout, SparkFun-Connectors:CONN_10X2
- added J2: (no value), SparkFun-Connectors:USB_MICRO-B_FEMALE-SMT
- added R2, R3: 10k, SparkFun-Resistors:10KOHM-0603-1/10W-1%
- added U$1: KMS231GLFS, KMS_Switches:KMS231GLFS
- added VD1: (no value), USBC6:USBLC6_USBLC6-2SC6
- added Y2: 32.768kHz, SparkFun-Clocks:CRYSTAL-32.768KHZSMD-3.2X1.5
- MCU: value STM32L052K8T -> MICRO-STM_V3_STM32L052K8T
Connections:
- new net N$2: C2.2, MCU.PC15-OSC_OUT, Y2.1
- new net N$3: C1.2, MCU.PC14-OSC_IN, Y2.2
- new net N$5: J2.D+, VD1.I/O_2
- new net N$6: J2.D-, VD1.I/O_1
- new net N$7: J2.VBUS, R2.1, VD1.VBUS
- new net N$8: MCU.PB1, R2.2, R3.1
- new net RESET: J1.5, MCU.NRST, U$1.1, U$1.5
- new net RX: J1.6, MCU.PB7
- new net SWCLK: J1.3, MCU.PA14
- new net SWDIO: J1.2, MCU.PA13
- new net TX: J1.4, MCU.PB6
- new net USB_DM: MCU.PA11, VD1.I/O1
- new net USB_DP: MCU.PA12, VD1.I/O2
- new net VDD: C3.1, C4.1, C5.1, J1.18
- new net VDDA: C6.1, C7.1, MCU.VDDA
- net GND: now also C1.1, C2.1, C3.2, C4.2, C5.2, C6.2, C7.2, J1.20, J2.GND, J2.SHIELD, R3.2, U$1.2, U$1.3, U$1.4, VD1.GND
- net N$1: now also MCU.BOOT0; no longer MCUMCU.BOOT0
Other:
- moved on the sheet: R1

Commit message: something
Parts:
- added 3V3REG: TLV76033DBZT, TLV76033DBZT:TLV76033DBZT
- added C8: 0.1uF, SparkFun-Capacitors:0.1UF-0603-25V-(+80/-20%)
- added C9: 1.0uF, SparkFun-Capacitors:1.0UF-0603-16V-10%
- MCU: value MICRO-STM_V3_STM32L052K8T -> STM32L052K8T
Connections:
- net N$8 renamed VBUS_DET
- removed net N$7: J2.VBUS, R2.1, VD1.VBUS
- new net +3V3: 3V3REG.OUT, C8.1
- new net VIN: 3V3REG.IN, C9.1, J1.18, J2.VBUS, R2.1, VD1.VBUS
- net GND: now also 3V3REG.GND, C8.2, C9.2, MCU.VSS@1, MCU.VSS@2
- net VDD: now also MCU.VDD@1, MCU.VDD@2; no longer J1.18
Other:
- moved on the sheet: C3, C4, C5, C6, C7
